Commit message: Various changes and fixes:
+ Updated models
+ Fixed py-bullet simulator, now embeds in GUI
+ Fixed py-bullet simulator crashing GUI when closing application forcefully

- Known bugs:
  - Imported objects are not resting on actuated platform
  - No controls are available in pybullet window

File: Data/sim/urdf/chamber.urdf (robot description, URDF)
Before this commit: robot chamber, 1 links, 0 joints
Links:
- removed link chamber
- added link chamber/frame; collision mesh filename=../Data/models/Chamber.obj scale=1 1 1; visual mesh filename=../Data/models/Chamber.obj scale=1 1 1
- added link chamber/world
Joints:
- added joint chamber/world_joint: type fixed, parent chamber/world, child chamber/frame, origin xyz=0 0 0 rpy=0 0 0

File: Data/sim/urdf/rx200pantex.urdf (robot description, URDF)
Before this commit: robot rx200pantex, 8 links, 7 joints
Links:
- removed link rx200pantex/base
- removed link rx200pantex/forearm_link
- removed link rx200pantex/mount
- removed link rx200pantex/probe_tip_ref
- removed link rx200pantex/shoulder_link
- removed link rx200pantex/upper_arm_link
- removed link rx200pantex/waist_link
- removed link rx200pantex/wrist_link
- added link rx200/base_link, mass 0.766135; collision mesh filename=../Data/sim/meshes/RX200_BASE.stl scale=0.001 0.001 0.001; visual mesh filename=../Data/sim/meshes/RX200_BASE.stl scale=0.001 0.001 0.001
- added link rx200/forearm_link, mass 0.258863; collision mesh filename=../Data/sim/meshes/RX200_FOREARM.stl scale=0.001 0.001 0.001; visual mesh filename=../Data/sim/meshes/RX200_FOREARM.stl scale=0.001 0.001 0.001
- added link rx200/linear_actuator, mass 20; collision mesh filename=../Data/sim/meshes/LINEAR_ACTUATOR.stl scale=0.001 0.001 0.001; visual mesh filename=../Data/sim/meshes/LINEAR_ACTUATOR.stl scale=0.001 0.001 0.001
- added link rx200/probe_tip_ref; collision sphere radius=0.005; visual sphere radius=0.005
- added link rx200/shoulder_link, mass 0.257774; collision mesh filename=../Data/sim/meshes/RX200_SHOULDER.stl scale=0.001 0.001 0.001; visual mesh filename=../Data/sim/meshes/RX200_SHOULDER.stl scale=0.001 0.001 0.001
- added link rx200/upper_arm_link, mass 0.297782; collision mesh filename=../Data/sim/meshes/RX200_UA.stl scale=0.001 0.001 0.001; visual mesh filename=../Data/sim/meshes/RX200_UA.stl scale=0.001 0.001 0.001
- added link rx200/wrist_link, mass 0.084957; collision mesh filename=../Data/sim/meshes/RX200_PROBE_WRIST.stl scale=0.001 0.001 0.001; visual mesh filename=../Data/sim/meshes/RX200_PROBE_WRIST.stl scale=0.001 0.001 0.001
- added link world
Joints:
- removed joint actuator_base_joint
- removed joint base_mount_joint
- added joint rail_base: type prismatic, parent rx200/linear_actuator, child rx200/base_link, origin xyz=0 -0.125 0.1425 rpy=0 0 0, axis 0 1 0, limit lower=0 upper=0.325 effort=8 velocity=0.05
- added joint world_joint: type fixed, parent world, child rx200/linear_actuator, origin xyz=0 0 0 rpy=0 0 0
- joint elbow: child rx200pantex/forearm_link -> rx200/forearm_link; limit lower=-1.8849555921538759 upper=1.6231562043547265 effort=1000 velocity=3.141592653589793 -> lower=-1.88496 upper=1.62316 effort=13 velocity=3.14159; parent rx200pantex/upper_arm_link -> rx200/upper_arm_link
- joint probe_ref_joint: child rx200pantex/probe_tip_ref -> rx200/probe_tip_ref; origin xyz=0.1475 0 0.0175 rpy=0 0 0 -> xyz=0.18 0.01 0.017 rpy=0 0 0; parent rx200pantex/wrist_link -> rx200/wrist_link
- joint shoulder: child rx200pantex/upper_arm_link -> rx200/upper_arm_link; limit lower=-1.8849555921538759 upper=1.9722220547535925 effort=1000 velocity=1 -> lower=-1.88496 upper=1.97222 effort=18 velocity=1; parent rx200pantex/shoulder_link -> rx200/shoulder_link
- joint waist: child rx200pantex/shoulder_link -> rx200/shoulder_link; limit lower=-3.141582653589793 upper=3.141582653589793 effort=8 velocity=3.141592653589793 -> lower=-1.57078632679 upper=1.57080632679 effort=8 velocity=3.14159; origin xyz=0 0 0.06566 rpy=0 0 0 -> xyz=0.00625 0 0 rpy=0 0 0; parent rx200pantex/waist_link -> rx200/base_link
- joint wrist_angle: child rx200pantex/wrist_link -> rx200/wrist_link; limit lower=-1.57079632679 upper=1.57079632679 effort=1000 velocity=3.141592653589793 -> lower=-1.74533 upper=2.14675 effort=5 velocity=3; parent rx200pantex/forearm_link -> rx200/forearm_link
