Commit message: fixed some UI stuff, added current slice to UI, working on dijkstras impl...

File: Data/sim/urdf/rx200pantex.urdf (robot description, URDF)
Before this commit: robot rx200, 8 links, 7 joints
Joints:
- joint probe_ref_joint: origin xyz=0.18 0.01 0.016 rpy=0 0 0 -> xyz=0.18 0.0075 0.016 rpy=0 0 0
