Commit message: created a way to set offsets!~

File: Data/sim/urdf/actuated_platform2.urdf (robot description, URDF)
Before this commit: robot actuated_platform, 3 links, 2 joints
Links:
- added link actuated_platform/object, mass 0.05; collision mesh filename=../Data/sim/meshes/object_exp.stl scale=0.001 0.001 0.001; visual mesh filename=../Data/sim/meshes/object_exp.stl scale=0.001 0.001 0.001
Joints:
- added joint object_plate_joint: type fixed, parent actuated_platform/plate, child actuated_platform/object, origin xyz=0.0 0.0 0.185
