Commit message: beginning force detection algorithm for force sensor

File: Data/sim/urdf/actuated_platform.urdf (robot description, URDF)
Before this commit: robot actuated_platform, 4 links, 3 joints
Joints:
- joint object_plate_joint: origin xyz=0.0 0.0 0.175 -> xyz=0.0 0.0 0.15875

Commit message: fully implemented NIDAQ - NIDAQ readings graphically available through 'info' on main GUI.

File: Data/sim/urdf/actuated_platform.urdf (robot description, URDF)
Before this commit: robot actuated_platform, 4 links, 3 joints
Joints:
- joint object_plate_joint: origin xyz=0.0 0.0 0.15875 -> xyz=0.0 0.0 0.175

Commit message: Updated robot controller, updated error handling

File: Data/sim/urdf/actuated_platform.urdf (robot description, URDF)
Before this commit: robot actuated_platform, 4 links, 3 joints
Joints:
- joint object_plate_joint: origin xyz=0.0 0.0 0.175 -> xyz=0.0 0.0 0.165

File: Data/sim/urdf/rx200pantex.urdf (robot description, URDF)
Before this commit: robot rx200, 8 links, 7 joints
Links:
- link rx200/linear_actuator: mass 20 -> 1
Joints:
- joint probe_ref_joint: origin xyz=0.18 0.01 0.017 rpy=0 0 0 -> xyz=0.18 0.01 0.016 rpy=0 0 0

Commit message: Implemented rectangular slicing

File: Data/sim/urdf/actuated_platform.urdf (robot description, URDF)
Before this commit: robot actuated_platform, 4 links, 3 joints
Joints:
- joint object_plate_joint: origin xyz=0.0 0.0 0.165 -> xyz=0.0 0.0 0.16

Commit message: grounding pause + object wizard stuff

File: Data/sim/urdf/actuated_platform.urdf (robot description, URDF)
Before this commit: robot actuated_platform, 4 links, 3 joints
Joints:
- joint object_plate_joint: origin xyz=0.0 0.0 0.16 -> xyz=0.0 0.0 0.175

Commit message: a bit of rectangular testing, closer to finished!

File: Data/sim/urdf/actuated_platform.urdf (robot description, URDF)
Before this commit: robot actuated_platform, 4 links, 3 joints
Joints:
- joint object_plate_joint: origin xyz=0.0 0.0 0.175 -> xyz=0.0 0.0 0.185

Commit message: So apparently, constrained objects lose the ability to be detected by a ray cast, so now im writing offsets to a new urdf that is used in the simulation!

File: Data/sim/urdf/actuated_platform.urdf (robot description, URDF)
Before this commit: robot actuated_platform, 3 links, 2 joints
Links:
- added link actuated_platform/object, mass 0.05; collision mesh filename=../Data/sim/meshes/object_exp.stl scale=0.001 0.001 0.001; visual mesh filename=../Data/sim/meshes/object_exp.stl scale=0.001 0.001 0.001
Joints:
- added joint object_plate_joint: type fixed, parent actuated_platform/plate, child actuated_platform/object, origin xyz=0.0 0.0 0.16

File: Data/sim/urdf/actuated_platform_no_obj.urdf (robot description, URDF)
Before this commit: robot actuated_platform, 4 links, 3 joints
Links:
- removed link actuated_platform/object
Joints:
- removed joint object_plate_joint

Commit message: home on termination / shutdown!

File: Data/sim/urdf/actuated_platform.urdf (robot description, URDF)
Before this commit: robot actuated_platform, 4 links, 3 joints
Joints:
- joint object_plate_joint: origin xyz=0.0 0.0 0.16 -> xyz=0.0 0.0 0.2

Commit message: Added a reduced main window since embedded pybullet wants to die!
also fixed probing alogrithm!

File: Data/sim/urdf/actuated_platform.urdf (robot description, URDF)
Before this commit: robot actuated_platform, 4 links, 3 joints
Joints:
- joint object_plate_joint: origin xyz=0.0 0.0 0.2 -> xyz=0.0 0.01 0.21000000000000002

Commit message: import obj done. adding config com port

File: Data/sim/urdf/actuated_platform.urdf (robot description, URDF)
Before this commit: robot actuated_platform, 4 links, 3 joints
Joints:
- joint object_plate_joint: origin xyz=0.0 0.01 0.21000000000000002 -> xyz=0.0 0.0 0.16

Commit message: fixes n thangs

File: Data/sim/urdf/actuated_platform.urdf (robot description, URDF)
Before this commit: robot actuated_platform, 4 links, 3 joints
Joints:
- joint object_plate_joint: origin xyz=0.0 0.0 0.16 -> xyz=0.0 0.0 0.176

Commit message: sometimes maybe good sometimes maybe shit

File: Data/sim/urdf/actuated_platform.urdf (robot description, URDF)
Before this commit: robot actuated_platform, 4 links, 3 joints
Joints:
- joint object_plate_joint: origin xyz=0.0 0.0 0.176 -> xyz=0.0 0.0 0.175

File: Data/sim/urdf/rx200pantex.urdf (robot description, URDF)
Before this commit: robot rx200, 8 links, 7 joints
Joints:
- joint probe_ref_joint: origin xyz=0.18 0.0075 0.016 rpy=0 0 0 -> xyz=0.155 0 0.016 rpy=0 0 0

Commit message: update

File: Data/sim/urdf/actuated_platform.urdf (robot description, URDF)
Before this commit: robot actuated_platform, 4 links, 3 joints
Joints:
- joint object_plate_joint: origin xyz=0.0 0.0 0.175 -> xyz=0.0 0.0 0.16
